Commit message: new_fast_neo

File: construct/src/environment/models/agent_models/neo.xacro (robot description, xacro)
@@ -8,8 +8,8 @@
 <xacro:property name="namespace" value="$(arg robot_namespace)" />
 <xacro:property name="use_mesh_file" value="true" />
-<xacro:property name="mesh_file" value="package://fcu_sim/meshes/Millennium_Falcon.dae" />
-<xacro:property name="mass" value="3.81" /> <!-- [kg] -->
-<xacro:property name="body_width" value="0.505" /> <!-- [m] -->
-<xacro:property name="body_height" value="0.1" /> <!-- [m] -->
+<xacro:property name="mesh_file" value="package://fcu_sim/meshes/firefly.dae" />
+<xacro:property name="mass" value="0.540" />
+<xacro:property name="body_width" value="0.3" />
+<xacro:property name="body_height" value="0.05" />
 <xacro:property name="rolling_moment_coefficient" value="0.000001" />
 <xacro:property name="body_inertia">
@@ -19,5 +19,5 @@
 <link name="${namespace}/base_link">
   <inertial>
-    <mass value="${mass}" />  <!-- [kg] -->
+    <mass value="${mass}" />
     <origin xyz="0 0 0" />
     <xacro:insert_block name="body_inertia" />
@@ -27,6 +27,5 @@
     <geometry>
       <xacro:if value="${use_mesh_file}">
-        <mesh filename="${mesh_file}" scale="0.001 0.001 0.001" />
-        <!-- <mesh filename="${mesh_file}" scale="1 1 1" /> -->
+        <mesh filename="${mesh_file}" scale="1 1 1" />
       </xacro:if>
       <xacro:unless value="${use_mesh_file}">
@@ -48,5 +47,5 @@
   <!-- Simplified Dynamics -->
   <xacro:include filename="$(find fcu_sim_plugins)/xacro/multirotor_forces_and_moments.xacro"/>
-  <xacro:mikey_forces_and_moments namespace="${namespace}" parent_link="${namespace}/base_link" command_topic="command"/>
+  <xacro:multirotor namespace="${namespace}" parent_link="${namespace}/base_link" command_topic="command"/>
   <!-- ***************** SENSORS ******************* -->
   <!-- Ground Truth -->
@@ -65,8 +64,7 @@
     image_camera_info_topic="camera_info">
     <origin xyz="0.127 0 -0.0889"/>
-    <!--<origin xyz="1 1 1"/>-->
   </xacro:step_camera>
   <!-- Laser Scanner -->
-  <xacro:include filename="$(find fcu_sim_plugins)/xacro/velodyne.xacro"/>
+<!--   <xacro:include filename="$(find fcu_sim_plugins)/xacro/velodyne.xacro"/>
   <xacro:velodyne_custom
     namespace="${namespace}"
@@ -76,24 +74,27 @@
     <origin xyz="${body_width+0.1} 0 0" rpy="0 0 0"/>
   </xacro:velodyne_custom>
+ -->
   <!-- GPS -->
-  <xacro:include filename="$(find fcu_sim_plugins)/xacro/GPS.xacro"/>
+<!--   <xacro:include filename="$(find fcu_sim_plugins)/xacro/GPS.xacro"/>
   <xacro:GPS_BYU
     namespace="${namespace}"
     parent_link="${namespace}/base_link"
     GPS_topic="gps"/>
+ -->
   <!-- Mount an IMU -->
-  <xacro:include filename="$(find fcu_sim_plugins)/xacro/imu.xacro"/>
+<!--   <xacro:include filename="$(find fcu_sim_plugins)/xacro/imu.xacro"/>
   <xacro:IMU_ADIS16448
     namespace="${namespace}"
     parent_link="${namespace}/base_link"
     imu_topic="imu"/>
+ -->
   <!-- Contact Sensor -->
-  <gazebo reference="${namespace}/base_link">
+<!--   <gazebo reference="${namespace}/base_link">
     <sensor name="contact_sensor" type="contact">
       <always_on>true</always_on>
       <update_rate>1000</update_rate>
       <contact>
-        <!-- When using ROS Indigo and Gazebo 2.2.3, the name specified here
-             must be <link name>_collision. -->
+        When using ROS Indigo and Gazebo 2.2.3, the name specified here
+             must be <link name>_collision.
         <collision>${namespace}/base_link_collision</collision>
       </contact>
@@ -104,3 +105,4 @@
     </sensor>
   </gazebo>
+ -->
 </robot>

Commit message: about to merge with james code

File: construct/src/environment/models/agent_models/neo.xacro (robot description, xacro)
@@ -5,45 +5,46 @@
 -->
 <robot name="neo" xmlns:xacro="http://ros.org/wiki/xacro">
-<!-- Properties -->
-<xacro:property name="namespace" value="$(arg robot_namespace)" />
-<xacro:property name="use_mesh_file" value="true" />
-<xacro:property name="mesh_file" value="package://fcu_sim/meshes/Millennium_Falcon.dae" />
-<xacro:property name="mass" value="3.81" /> <!-- [kg] -->
-<xacro:property name="body_width" value="0.505" /> <!-- [m] -->
-<xacro:property name="body_height" value="0.1" /> <!-- [m] -->
-<xacro:property name="rolling_moment_coefficient" value="0.000001" />
-<xacro:property name="body_inertia">
-  <inertia ixx="0.0347563" ixy="0.0" ixz="0.0" iyy="0.0458929" iyz="0.0" izz="0.0977" />
-</xacro:property>
-<!-- *********************** GAZEBO ROBOT DEFINITION ******************* -->
-<link name="${namespace}/base_link">
-  <inertial>
-    <mass value="${mass}" />  <!-- [kg] -->
-    <origin xyz="0 0 0" />
-    <xacro:insert_block name="body_inertia" />
-  </inertial>
-  <visual>
-    <origin xyz="0 0 0" rpy="0 0 0" />
-    <geometry>
-      <xacro:if value="${use_mesh_file}">
-        <mesh filename="${mesh_file}" scale="0.001 0.001 0.001" />
-        <!-- <mesh filename="${mesh_file}" scale="1 1 1" /> -->
-      </xacro:if>
-      <xacro:unless value="${use_mesh_file}">
+  <!-- Properties -->
+  <xacro:property name="namespace" value="neo" />
+  <xacro:property name="use_mesh_file" value="true" />
+  <xacro:property name="mesh_file" value="package://fcu_sim/meshes/firefly.dae" />
+  <xacro:property name="mass" value="3.562" />
+  <xacro:property name="body_width" value="0.505" />
+  <xacro:property name="body_height" value="0.1" />
+  <xacro:property name="body_inertia">
+    <inertia ixx="0.0347563" ixy="0.0" ixz="0.0" iyy="0.0458929" iyz="0.0" izz="0.0977" />
+  </xacro:property>
+  <!-- *********************** GAZEBO ROBOT DEFINITION ******************* -->
+  <link name="${namespace}/base_link">
+    <inertial>
+      <mass value="${mass}" />  <!-- [kg] -->
+      <origin xyz="0 0 0" />
+      <xacro:insert_block name="body_inertia" />
+    </inertial>
+    <visual>
+      <origin xyz="0 0 0" rpy="0 0 0" />
+      <geometry>
+        <xacro:if value="${use_mesh_file}">
+          <mesh filename="${mesh_file}" scale="1 1 1" />
+        </xacro:if>
+        <xacro:unless value="${use_mesh_file}">
+          <cylinder length="${body_height}" radius="${body_width}"/>
+        </xacro:unless>
+      </geometry>
+    </visual>
+    <collision>
+      <origin xyz="0 0 0" rpy="0 0 0" />
+      <geometry>
         <cylinder length="${body_height}" radius="${body_width}"/>
-      </xacro:unless>
-    </geometry>
-  </visual>
-  <collision name="collision_mav">
-    <origin xyz="0 0 ${body_height/2.0}" rpy="0 0 0" />
-    <geometry>
-      <cylinder length="${0.1}" radius="${body_width}"/>
-    </geometry>
-  </collision>
-</link>
+      </geometry>
+    </collision>
+  </link>
   <gazebo reference="${namespace}/base_link">
     <material>Gazebo/$(arg color)</material>
   </gazebo>
   <!-- ************************* ROTOR DYNAMICS ********************** -->
+  <!-- ROSflight_SIL
+  <xacro:include filename="$(find fcu_sim_plugins)/xacro/ROSflight_SIL.xacro"/>
+  <xacro:mikey_ROSflight_SIL namespace="${namespace}" parent_link="${namespace}/base_link" command_topic="command"/> -->
   <!-- Simplified Dynamics -->
   <xacro:include filename="$(find fcu_sim_plugins)/xacro/multirotor_forces_and_moments.xacro"/>
@@ -65,5 +66,4 @@
     image_camera_info_topic="camera_info">
     <origin xyz="0.127 0 -0.0889"/>
-    <!--<origin xyz="1 1 1"/>-->
   </xacro:step_camera>
   <!-- Laser Scanner -->
@@ -94,6 +94,4 @@
       <update_rate>1000</update_rate>
       <contact>
-        <!-- When using ROS Indigo and Gazebo 2.2.3, the name specified here
-             must be <link name>_collision. -->
         <collision>${namespace}/base_link_collision</collision>
       </contact>

Commit message: still trying to get everything working

File: construct/src/environment/models/agent_models/neo.xacro (robot description, xacro)
@@ -6,5 +6,5 @@
 <robot name="neo" xmlns:xacro="http://ros.org/wiki/xacro">
 <!-- Properties -->
-<xacro:property name="namespace" value="neo" />
+<xacro:property name="namespace" value="$(arg robot_namespace)" />
 <xacro:property name="use_mesh_file" value="true" />
 <xacro:property name="mesh_file" value="package://fcu_sim/meshes/firefly.dae" />
@@ -31,14 +31,18 @@
       <xacro:unless value="${use_mesh_file}">
         <cylinder length="${body_height}" radius="${body_width}"/>
-      </geometry>
-    </collision>
-  </link>
+      </xacro:unless>
+    </geometry>
+  </visual>
+  <collision name="collision_mav">
+    <origin xyz="0 0 ${body_height/2.0}" rpy="0 0 0" />
+    <geometry>
+      <cylinder length="${0.1}" radius="${body_width}"/>
+    </geometry>
+  </collision>
+</link>
   <gazebo reference="${namespace}/base_link">
     <material>Gazebo/$(arg color)</material>
   </gazebo>
   <!-- ************************* ROTOR DYNAMICS ********************** -->
-  <!-- ROSflight_SIL
-  <xacro:include filename="$(find fcu_sim_plugins)/xacro/ROSflight_SIL.xacro"/>
-  <xacro:mikey_ROSflight_SIL namespace="${namespace}" parent_link="${namespace}/base_link" command_topic="command"/> -->
   <!-- Simplified Dynamics -->
   <xacro:include filename="$(find fcu_sim_plugins)/xacro/multirotor_forces_and_moments.xacro"/>
@@ -79,11 +83,10 @@
  -->
   <!-- Mount an IMU -->
-<!--   <xacro:include filename="$(find fcu_sim_plugins)/xacro/imu.xacro"/>
+  <xacro:include filename="$(find fcu_sim_plugins)/xacro/imu.xacro"/>
   <xacro:IMU_ADIS16448
     namespace="${namespace}"
     parent_link="${namespace}/base_link"
     imu_topic="imu"/>
- -->
-  <!-- Contact Sensor
+  <!-- Contact Sensor -->
   <gazebo reference="${namespace}/base_link">
     <sensor name="contact_sensor" type="contact">
@@ -98,4 +101,4 @@
       </plugin>
     </sensor>
-  </gazebo>-->
+  </gazebo>
 </robot>

Commit message: collision fixed for gazebo7

File: construct/src/environment/models/agent_models/neo.xacro (robot description, xacro)
@@ -27,5 +27,6 @@
     <geometry>
       <xacro:if value="${use_mesh_file}">
-        <mesh filename="${mesh_file}" scale="1 1 1" />
+        <cylinder length="${body_height}" radius="${body_width}"/>
+        <!--<mesh filename="${mesh_file}" scale="1 1 1" />-->
       </xacro:if>
       <xacro:unless value="${use_mesh_file}">
@@ -34,8 +35,8 @@
     </geometry>
   </visual>
-  <collision name="collision_mav">
-    <origin xyz="0 0 ${body_height/2.0}" rpy="0 0 0" />
+  <collision name="mav_collision">
+    <origin xyz="0 0 0" rpy="0 0 0" />
     <geometry>
-      <cylinder length="${0.1}" radius="${body_width}"/>
+      <cylinder length="${body_height}" radius="${body_width}"/>
     </geometry>
   </collision>
@@ -52,5 +53,5 @@
   <xacro:include filename="$(find fcu_sim_plugins)/xacro/odometry_sensor.xacro"/>
   <xacro:ground_truth namespace="${namespace}" parent_link="${namespace}/base_link" />
-  <!-- Step Camera -->
+  <!-- Step Camera  -->
   <xacro:include filename="$(find fcu_sim_plugins)/xacro/step_camera.xacro"/>
   <xacro:step_camera
@@ -82,17 +83,26 @@
     GPS_topic="gps"/>
  -->
-  <!-- Mount an IMU -->
+  <!-- Mount an IMU
   <xacro:include filename="$(find fcu_sim_plugins)/xacro/imu.xacro"/>
   <xacro:IMU_ADIS16448
     namespace="${namespace}"
     parent_link="${namespace}/base_link"
-    imu_topic="imu"/>
+    imu_topic="imu"/> -->
   <!-- Contact Sensor -->
   <gazebo reference="${namespace}/base_link">
     <sensor name="contact_sensor" type="contact">
       <always_on>true</always_on>
-      <update_rate>1000</update_rate>
+      <update_rate>100</update_rate>
       <contact>
-        <collision>${namespace}/base_link_collision</collision>
+        <!-- Probably one of the ugliest bugs I've seen in Gazebo: http://answers.gazebosim.org/question/15095/gazebo-contact-sensor-added-to-a-robot-link-in-urdf-file-is-not-working-as-expected/
+         There is an error in the conversion from xacro -> URDF -> SDF that creates default
+         collision names
+        -->
+        <collision>${namespace}/base_link_fixed_joint_lump__mav_collision_collision</collision>
+        <!-- In older versions of Gazebo:
+          <contact>
+            <collision>${namespace}/base_link_collision</collision>
+          </contact>
+        -->
       </contact>
       <plugin name="fixed_jaw_bumper" filename="libgazebo_ros_bumper.so">

Commit message: about to delete multiworldmanager

File: construct/src/environment/models/agent_models/neo.xacro (robot description, xacro)
@@ -27,6 +27,5 @@
     <geometry>
       <xacro:if value="${use_mesh_file}">
-        <cylinder length="${body_height}" radius="${body_width}"/>
-        <!--<mesh filename="${mesh_file}" scale="1 1 1" />-->
+        <mesh filename="${mesh_file}" scale="1 1 1" />
       </xacro:if>
       <xacro:unless value="${use_mesh_file}">
@@ -93,5 +92,5 @@
     <sensor name="contact_sensor" type="contact">
       <always_on>true</always_on>
-      <update_rate>100</update_rate>
+      <update_rate>10</update_rate>
       <contact>
         <!-- Probably one of the ugliest bugs I've seen in Gazebo: http://answers.gazebosim.org/question/15095/gazebo-contact-sensor-added-to-a-robot-link-in-urdf-file-is-not-working-as-expected/

Commit message: added CEPA, tested plumbing, things look pretty much right

File: construct/src/environment/models/agent_models/neo.xacro (robot description, xacro)
@@ -54,6 +54,6 @@
   <!-- Step Camera -->
   <!-- The width and/or height MUST remain larger than 255 in order to ues faster-than-real-time: https://bitbucket.org/osrf/gazebo/issues/2214/width-height-255-for-camera-causes -->
-  <xacro:include filename="$(find fcu_sim_plugins)/xacro/step_camera.xacro"/>
-  <xacro:step_camera
+  <!-- <xacro:include filename="$(find fcu_sim_plugins)/xacro/step_camera.xacro"/> -->
+<!--   <xacro:step_camera
     namespace="${namespace}"
     frame_rate="25"
@@ -65,15 +65,15 @@
     image_camera_info_topic="camera_info">
     <origin xyz="0.127 0 -0.0889"/>
-  </xacro:step_camera>
+  </xacro:step_camera>  -->
   <!-- Laser Scanner -->
-<!--   <xacro:include filename="$(find fcu_sim_plugins)/xacro/velodyne.xacro"/>
-  <xacro:velodyne_custom
+  <xacro:include filename="gimbal_laser.xacro"/>
+  <!-- <xacro:include filename="$(find fcu_sim_plugins)/xacro/laser_scanner.xacro"/> -->
+  <xacro:gimbal_laser
     namespace="${namespace}"
     parent_link="${namespace}/base_link"
-    update_rate="25"
-    visualize="false">
-    <origin xyz="${body_width+0.1} 0 0" rpy="0 0 0"/>
-  </xacro:velodyne_custom>
- -->
+    visualize="false"
+    pose_topic="laser_pose">
+    <origin xyz="0 0 ${body_height+1.0}" rpy="0 0 0"/>
+  </xacro:gimbal_laser>
   <!-- GPS -->
 <!--   <xacro:include filename="$(find fcu_sim_plugins)/xacro/GPS.xacro"/>
