Commit message: added random world

File: construct/src/environment/models/agent_models/gimbal_laser.xacro (robot description, xacro)
@@ -15,7 +15,7 @@
       visualize="${visualize}"
       mass="0.00001"
-      x_rotation_range="1000000000"
-      y_rotation_range="1000000000"
-      z_rotation_range="1000000000"
+      x_rotation_range="1000"
+      y_rotation_range="1000"
+      z_rotation_range="1000"
       time_constant="0.00001">
       <inertia ixx="0.00001" ixy="0.0" ixz="0.0" iyy="0.00001" iyz="0.0" izz="0.00001" />
@@ -28,5 +28,4 @@
     params="namespace parent_link pose_topic visualize mass x_rotation_range
             y_rotation_range z_rotation_range time_constant *inertia *origin">
-    <!-- Base Link  -->
     <link name="${namespace}/gimbal/base_link">
       <inertial>
@@ -36,5 +35,4 @@
       </inertial>
     </link>
-    <!-- Base Joint -->
     <joint name="${namespace}/gimbal_base_joint" type="revolute">
       <xacro:insert_block name="origin" />
@@ -43,5 +41,4 @@
       <limit upper="0" lower="0" effort="0" velocity="0"/>
     </joint>
-    <!-- Yaw Link -->
     <link name="${namespace}/gimbal/yaw_link">
       <inertial>
@@ -51,5 +48,4 @@
       </inertial>
     </link>
-    <!-- Yaw joint -->
     <joint name="${namespace}/gimbal_yaw_joint" type="revolute">
       <pose xyz="0 0 0" rpy = "0 0 0"/>
@@ -58,5 +54,4 @@
       <limit upper="${z_rotation_range}" lower="${-1.0*z_rotation_range}" effort="1000" velocity="5000"/>
     </joint>
-    <!-- Pitch Link -->
     <link name="${namespace}/gimbal/pitch_link">
       <inertial>
@@ -66,5 +61,4 @@
       </inertial>
     </link>
-    <!-- Pitch joint -->
     <joint name="${namespace}/gimbal_pitch_joint" type="revolute">
       <origin xyz="0 0 0" rpy = "0 0 0"/>
@@ -73,5 +67,4 @@
       <limit upper="${x_rotation_range}" lower="${-1.0*x_rotation_range}" effort="1000" velocity="5000"/>
     </joint>
-        <!-- Roll Link -->
     <link name="${namespace}/gimbal/roll_link">
       <inertial>
@@ -81,5 +74,4 @@
       </inertial>
     </link>
-    <!-- Roll joint -->
     <joint name="${namespace}/gimbal_roll_joint" type="revolute">
       <origin xyz="0 0 0" rpy = "0 0 0"/>
@@ -88,45 +80,37 @@
       <limit upper="${x_rotation_range}" lower="${-1.0*x_rotation_range}" effort="1000" velocity="5000"/>
     </joint>
-    <!-- Attach a Camera -->
-<!--     <gazebo reference="${namespace}/gimbal/pitch_link">
-      <sensor type="camera" name="gimbal/camera">
-        <always_on>true</always_on>
-	<update_rate>${frame_rate}</update_rate>
-        <camera>
-          <horizontal_fov>2</horizontal_fov>
-          <image>
-            <format>R8G8B8</format>
-            <width>640</width>
-            <height>480</height>
-          </image>
-          <clip>
-            <near>0.01</near>
-            <far>1000</far>
-          </clip>
-        </camera>
-	<plugin filename="libfcu_sim_camera_plugin.so" name="${namespace}/gimbal_camera">
-          <robotNamespace>${namespace}</robotNamespace>
-          <alwaysOn>true</alwaysOn>
-	  <updateRate>${frame_rate}</updateRate>
-          <cameraName>gimbal/camera</cameraName>
-          <imageTopicName>${camera_topic}</imageTopicName>
-          <cameraInfoTopicName>${camera_topic}/camera_info</cameraInfoTopicName>
-          <frameName>gimbal_camera</frameName>
-          <distortionK1>0.0</distortionK1>
-          <distortionK2>0.0</distortionK2>
-          <distortionK3>0.0</distortionK3>
-          <distortionT1>0.0</distortionT1>
-          <distortionT2>0.0</distortionT2>
-        </plugin>
-      </sensor>
-    </gazebo> -->
     <!-- Attach a Laser Scanner -->
-    <xacro:include filename="$(find fcu_sim_plugins)/xacro/laser_scanner.xacro"/>
-    <xacro:RPLIDAR-A2
-      namespace="${namespace}"
-      parent_link="${namespace}/gimbal/roll_link"
-      visualize="${visualize}">
-      <origin xyz="0 0 0.5" rpy="0 0 0"/>
-    </xacro:RPLIDAR-A2>
+    <gazebo reference="${namespace}/gimbal/base_link">
+    <sensor type="ray" name="laser_scanner">
+      <pose>0 0 0 0 0 0</pose>
+      <visualize>false</visualize>
+      <update_rate>1</update_rate>
+      <ray>
+        <scan>
+          <horizontal>
+            <samples>720</samples>
+            <resolution>1</resolution>
+            <min_angle>-3.14159</min_angle>
+            <max_angle>3.14159</max_angle>
+          </horizontal>
+        </scan>
+        <range>
+          <min>0.10</min>
+          <max>30.0</max>
+          <resolution>0.01</resolution>
+        </range>
+        <noise>
+          <type>gaussian</type>
+          <mean>0.0</mean>
+          <stddev>0.01</stddev>
+        </noise>
+      </ray>
+      <plugin name="${namespace}_laser" filename="libgazebo_ros_laser.so">
+        <topicName>${namespace}/scan</topicName>
+        <frameName>${namespace}/
+        </frameName>
+      </plugin>
+    </sensor>
+  </gazebo>
     <!-- Load Gimbal Controller Plugin -->
     <gazebo>

File: construct/src/environment/models/agent_models/neo.xacro (robot description, xacro)
@@ -53,7 +53,7 @@
   <xacro:ground_truth namespace="${namespace}" parent_link="${namespace}/base_link" />
   <!-- Step Camera -->
-  <!-- The width and/or height MUST remain larger than 255 in order to ues faster-than-real-time: https://bitbucket.org/osrf/gazebo/issues/2214/width-height-255-for-camera-causes -->
-  <!-- <xacro:include filename="$(find fcu_sim_plugins)/xacro/step_camera.xacro"/> -->
-<!--   <xacro:step_camera
+  <!-- The width and/or height MUST remain larger than 255 in order to ues faster-than-real-time: https://bitbucket.org/osrf/gazebo/issues/2214/width-height-255-for-camera-causes  -->
+  <xacro:include filename="$(find fcu_sim_plugins)/xacro/step_camera.xacro"/>
+   <xacro:step_camera
     namespace="${namespace}"
     frame_rate="25"
@@ -65,8 +65,7 @@
     image_camera_info_topic="camera_info">
     <origin xyz="0.127 0 -0.0889"/>
-  </xacro:step_camera>  -->
+  </xacro:step_camera>
   <!-- Laser Scanner -->
   <xacro:include filename="gimbal_laser.xacro"/>
-  <!-- <xacro:include filename="$(find fcu_sim_plugins)/xacro/laser_scanner.xacro"/> -->
   <xacro:gimbal_laser
     namespace="${namespace}"

Commit message: now working with new obstacle avoidance

File: construct/src/environment/models/agent_models/gimbal_laser.xacro (robot description, xacro)
@@ -28,104 +28,85 @@
     params="namespace parent_link pose_topic visualize mass x_rotation_range
             y_rotation_range z_rotation_range time_constant *inertia *origin">
+  <gazebo>
     <link name="${namespace}/gimbal/base_link">
       <inertial>
-        <inertia ixx="0.00001" ixy="0.0" ixz="0.0" iyy="0.00001" iyz="0.0" izz="0.00001" />
-        <mass value="${mass}" />
-        <xacro:insert_block name="origin" />
+          <inertia>
+              <ixx>0.000</ixx>
+              <ixy>0.000</ixy>
+              <ixz>0.000</ixz>
+              <iyy>0.000</iyy>
+              <iyz>0.000</iyz>
+              <izz>0.000</izz>
+          </inertia>
+          <mass>${mass}</mass>
       </inertial>
+      <pose>0 0 -.50 0 0 0</pose>
+      <sensor type="ray" name="laser_scanner">
+        <pose>0 0 0 0 0 0</pose>
+        <visualize>true</visualize>
+        <update_rate>25</update_rate>
+        <ray>
+          <scan>
+            <horizontal>
+              <samples>720</samples>
+              <resolution>1</resolution>
+              <min_angle>-3.14159</min_angle>
+              <max_angle>3.14159</max_angle>
+            </horizontal>
+          </scan>
+          <range>
+            <min>0.10</min>
+            <max>30.0</max>
+            <resolution>0.01</resolution>
+          </range>
+          <noise>
+            <type>gaussian</type>
+            <mean>0.0</mean>
+            <stddev>0.01</stddev>
+          </noise>
+        </ray>
+        <plugin name="${namespace}_laser" filename="libgazebo_ros_laser.so">
+          <topicName>${namespace}/scan</topicName>
+          <frameName>${namespace}/</frameName>
+        </plugin>
+      </sensor>
     </link>
-    <joint name="${namespace}/gimbal_base_joint" type="revolute">
-      <xacro:insert_block name="origin" />
-      <parent link="${parent_link}" />
-      <child link="${namespace}/gimbal/base_link" />
-      <limit upper="0" lower="0" effort="0" velocity="0"/>
+    <joint name="${namespace}/gimbal_base_joint" type="ball">
+      <parent>${parent_link}</parent>
+      <child>${namespace}/gimbal/base_link</child>
     </joint>
-    <link name="${namespace}/gimbal/yaw_link">
-      <inertial>
-        <inertia ixx="0.00001" ixy="0.0" ixz="0.0" iyy="0.00001" iyz="0.0" izz="0.00001" />
-        <mass value="${mass}" />
-        <origin xyz="0 0 0" rpy = "0 0 0"/>
-      </inertial>
-    </link>
-    <joint name="${namespace}/gimbal_yaw_joint" type="revolute">
-      <pose xyz="0 0 0" rpy = "0 0 0"/>
-      <parent link="${namespace}/gimbal/base_link" />
-      <child link="${namespace}/gimbal/yaw_link" />
-      <limit upper="${z_rotation_range}" lower="${-1.0*z_rotation_range}" effort="1000" velocity="5000"/>
-    </joint>
-    <link name="${namespace}/gimbal/pitch_link">
-      <inertial>
-        <inertia ixx="0.00001" ixy="0.0" ixz="0.0" iyy="0.00001" iyz="0.0" izz="0.00001" />
-        <mass value="${mass}" />
-        <origin xyz="0 0 0" rpy = "0 0 0"/>
-      </inertial>
-    </link>
-    <joint name="${namespace}/gimbal_pitch_joint" type="revolute">
-      <origin xyz="0 0 0" rpy = "0 0 0"/>
-      <parent link="${namespace}/gimbal/yaw_link" />
-      <child link="${namespace}/gimbal/pitch_link" />
-      <limit upper="${x_rotation_range}" lower="${-1.0*x_rotation_range}" effort="1000" velocity="5000"/>
-    </joint>
-    <link name="${namespace}/gimbal/roll_link">
-      <inertial>
-        <inertia ixx="0.00001" ixy="0.0" ixz="0.0" iyy="0.00001" iyz="0.0" izz="0.00001" />
-        <mass value="${mass}" />
-        <origin xyz="0 0 0" rpy = "0 0 0"/>
-      </inertial>
-    </link>
-    <joint name="${namespace}/gimbal_roll_joint" type="revolute">
-      <origin xyz="0 0 0" rpy = "0 0 0"/>
-      <parent link="${namespace}/gimbal/pitch_link" />
-      <child link="${namespace}/gimbal/roll_link" />
-      <limit upper="${x_rotation_range}" lower="${-1.0*x_rotation_range}" effort="1000" velocity="5000"/>
-    </joint>
-    <!-- Attach a Laser Scanner -->
-    <gazebo reference="${namespace}/gimbal/base_link">
-    <sensor type="ray" name="laser_scanner">
-      <pose>0 0 0 0 0 0</pose>
-      <visualize>false</visualize>
-      <update_rate>1</update_rate>
-      <ray>
-        <scan>
-          <horizontal>
-            <samples>720</samples>
-            <resolution>1</resolution>
-            <min_angle>-3.14159</min_angle>
-            <max_angle>3.14159</max_angle>
-          </horizontal>
-        </scan>
-        <range>
-          <min>0.10</min>
-          <max>30.0</max>
-          <resolution>0.01</resolution>
-        </range>
-        <noise>
-          <type>gaussian</type>
-          <mean>0.0</mean>
-          <stddev>0.01</stddev>
-        </noise>
-      </ray>
-      <plugin name="${namespace}_laser" filename="libgazebo_ros_laser.so">
-        <topicName>${namespace}/scan</topicName>
-        <frameName>${namespace}/
-        </frameName>
-      </plugin>
-    </sensor>
+    <plugin filename="libautolevel_plugin.so" name="fcu_sim_gimbal_plugin">
+        <namespace>${namespace}</namespace>
+        <sensorLink>${namespace}/gimbal/base_link</sensorLink>
+        <modelLink>${parent_link}</modelLink>
+    </plugin>
   </gazebo>
-    <!-- Load Gimbal Controller Plugin -->
-    <gazebo>
-      <plugin filename="libgimbal_plugin.so" name="fcu_sim_gimbal_plugin">
-        <namespace>${namespace}</namespace>
-        <yawJoint>${namespace}/gimbal_yaw_joint</yawJoint>
-        <pitchJoint>${namespace}/gimbal_pitch_joint</pitchJoint>
-        <rollJoint>${namespace}/gimbal_roll_joint</rollJoint>
-        <timeConstant>${time_constant}</timeConstant>
-        <commandTopic>empty</commandTopic>
-        <poseTopic>${pose_topic}</poseTopic>
-        <useSlipring>true</useSlipring>
-        <linkName>${parent_link}</linkName>
-        <autoStabilize>true</autoStabilize>
-      </plugin>
-    </gazebo>
+  <!--<gazebo>-->
+  <!--<link name="${namespace}\ball_link">-->
+      <!--<gravity>1</gravity>-->
+      <!--&lt;!&ndash; Put the ball just under the socket &ndash;&gt;-->
+      <!--<pose >0.4 0 0.35 0 0 0</pose>-->
+      <!--<inertial>-->
+          <!--<mass>0.0001</mass> &lt;!&ndash; kg &ndash;&gt;-->
+          <!--<inertia>-->
+              <!--&lt;!&ndash; (2 * mass * radius * radius) / 5 &ndash;&gt;-->
+              <!--<ixx>0.00196</ixx>-->
+              <!--&lt;!&ndash; fudge it a bit to get movement on two axis from gravity alone &ndash;&gt;-->
+              <!--<ixy>0.001</ixy>-->
+              <!--<ixz>0.001</ixz>-->
+              <!--&lt;!&ndash; (2 * mass * radius * radius) / 5 &ndash;&gt;-->
+              <!--<iyy>0.00196</iyy>-->
+              <!--<iyz>0.001</iyz>-->
+              <!--&lt;!&ndash; (2 * mass * radius * radius) / 5 &ndash;&gt;-->
+              <!--<izz>0.00196</izz>-->
+          <!--</inertia>-->
+          <!--&lt;!&ndash; offset interia as a trick to get movement from gravity &ndash;&gt;-->
+          <!--<pose >0.1 -0.1 0.1 0 0 0</pose>-->
+      <!--</inertial>-->
+  <!--</link>-->
+  <!--<joint name="${namespace}\ball_joint" type="ball">-->
+      <!--<parent>${parent_link}</parent>-->
+      <!--<child>${namespace}\ball_link</child>-->
+  <!--</joint>-->
   </xacro:macro>
 </robot>
